Commit message: .

File: arm_description/urdf/Kikobot.urdf (robot description, URDF)
Before this commit: robot Kikobot, 8 links, 7 joints
Links:
- link Arm-1: geometry collision mesh filename=package://arm_description/urdf/meshes/Arm-1.stl scale=0.001 0.001 0.001; visual mesh filename=package://arm_description/urdf/meshes/Arm-1.stl scale=0.001 0.001 0.001
- link Arm-2: geometry collision mesh filename=package://arm_description/urdf/meshes/Arm-2.stl scale=0.001 0.001 0.001; visual mesh filename=package://arm_description/urdf/meshes/Arm-2.stl scale=0.001 0.001 0.001
- link Arm-3: geometry collision mesh filename=package://arm_description/urdf/meshes/Arm-3.stl scale=0.001 0.001 0.001; visual mesh filename=package://arm_description/urdf/meshes/Arm-3.stl scale=0.001 0.001 0.001
- link Arm-4: geometry collision mesh filename=package://arm_description/urdf/meshes/Arm-4.stl scale=0.001 0.001 0.001; visual mesh filename=package://arm_description/urdf/meshes/Arm-4.stl scale=0.001 0.001 0.001
- link Arm-5: geometry collision mesh filename=package://arm_description/urdf/meshes/Arm-5.stl scale=0.001 0.001 0.001; visual mesh filename=package://arm_description/urdf/meshes/Arm-5.stl scale=0.001 0.001 0.001
- link Base: geometry collision mesh filename=package://arm_description/urdf/meshes/Base.stl scale=0.001 0.001 0.001; visual mesh filename=package://arm_description/urdf/meshes/Base.stl scale=0.001 0.001 0.001
- link End-Coupler-v1: geometry collision mesh filename=package://arm_description/urdf/meshes/End-Coupler-v1.stl scale=0.001 0.001 0.001; visual mesh filename=package://arm_description/urdf/meshes/End-Coupler-v1.stl scale=0.001 0.001 0.001
