Commit message: Updated Readme with Physics Properties

File: arm_description/urdf/arm.urdf.xacro (robot description, xacro)
@@ -166,5 +166,6 @@
     <child link="Arm-1" />
     <axis xyz="0.0 0.0 1.0" />
-    <limit lower="-2.879793" upper="2.879793" effort="1000000" velocity="1000000" />
+    <limit lower="-2.879793" upper="2.879793" effort="150.0" velocity="2.0" />
+    <dynamics damping="0.8" friction="0.5" />
   </joint>
   <joint name="Arm-1_Revolute-2" type="revolute">
@@ -173,5 +174,6 @@
     <child link="Arm-2" />
     <axis xyz="1.0 8.531573731886488e-33 0.0" />
-    <limit lower="-2.181662" upper="2.181662" effort="1000000" velocity="1000000" />
+    <limit lower="-2.181662" upper="2.181662" effort="120.0" velocity="1.8" />
+    <dynamics damping="0.6" friction="0.4" />
   </joint>
   <joint name="Arm-2_Revolute-3" type="revolute">
@@ -180,5 +182,6 @@
     <child link="Arm-3" />
     <axis xyz="0.0 0.0 -1.0" />
-    <limit lower="-2.443461" upper="2.443461" effort="1000000" velocity="1000000" />
+    <limit lower="-2.443461" upper="2.443461" effort="80.0" velocity="2.5" />
+    <dynamics damping="0.4" friction="0.3" />
   </joint>
   <joint name="Arm-3_Revolute-4" type="revolute">
@@ -187,5 +190,6 @@
     <child link="Arm-4" />
     <axis xyz="1.232595164407831e-32 -1.9721522630525295e-31 1.0" />
-    <limit lower="-2.443461" upper="2.443461" effort="1000000" velocity="1000000" />
+    <limit lower="-2.443461" upper="2.443461" effort="40.0" velocity="3.0" />
+    <dynamics damping="0.3" friction="0.2" />
   </joint>
   <joint name="Arm-4_Revolute-5" type="revolute">
@@ -194,5 +198,6 @@
     <child link="Arm-5" />
     <axis xyz="0.0 1.0 0.0" />
-    <limit lower="-2.443461" upper="2.443461" effort="1000000" velocity="1000000" />
+    <limit lower="-2.443461" upper="2.443461" effort="25.0" velocity="3.5" />
+    <dynamics damping="0.2" friction="0.15" />
   </joint>
   <joint name="Arm-5_Revolute-6" type="revolute">
@@ -201,5 +206,6 @@
     <child link="End-Coupler-v1" />
     <axis xyz="-1.0 -9.679619902524347e-33 -0.0" />
-    <limit lower="-3.054326" upper="3.054326" effort="1000000" velocity="1000000" />
+    <limit lower="-3.054326" upper="3.054326" effort="15.0" velocity="4.0" />
+    <dynamics damping="0.1" friction="0.1" />
   </joint>
   <ros2_control name="KikobotSystem" type="system">

Commit message: minor changes in URDF

File: arm_description/urdf/arm.urdf.xacro (robot description, xacro)
@@ -1,3 +1,3 @@
-<robot name="Kikobot">
+<robot name="robo_arm">
   <link name="world" />
   <material name="ur_accent">
@@ -14,5 +14,17 @@
     <parent link="world" />
     <child link="base_link" />
-    <origin xyz="0 0 0" rpy="0 0 0" />
+    <origin xyz="0 0 0" rpy="0 0 0" />    <ros2_control name="KikobotSystem" type="system">
+      <hardware>
+        <plugin>gz_ros2_control/GazeboSimSystem</plugin>
+      </hardware>
+      <joint name="...">...</joint>
+      ...
+    </ros2_control>    <ros2_control name="KikobotSystem" type="system">
+      <hardware>
+        <plugin>gz_ros2_control/GazeboSimSystem</plugin>
+      </hardware>
+      <joint name="...">...</joint>
+      ...
+    </ros2_control>
   </joint>
   <joint name="base_link_to_Base" type="fixed">
@@ -209,5 +221,5 @@
     <dynamics damping="0.1" friction="0.1" />
   </joint>
-  <ros2_control name="KikobotSystem" type="system">
+  <ros2_control name="RobotSystem" type="system">
     <hardware>
       <plugin>gz_ros2_control/GazeboSimSystem</plugin>
